File: hardware/MSP430Geiger/MSP430Geiger.brd (EAGLE design)
At the start: 90.3 x 90.2 mm, 84 parts, among them IC1 LDO, IC2 MSP430, IC3 LM555D, IC4 LM555N, IC5 LM321MF, Q1 2N2222, Q2 MPSA42, Q3 2N2222, T1 DMN3024LSD, T2 2N2222(N.M)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

Commit message: edit
Parts:
- added C13: 10uF, SparkFun-Capacitors:0603-CAP
Connections:
- net GND: now also C13.2
- net VDD: now also C13.1
Routing:
- net VDD: track 260.3 -> 266.8 mm
- net GND: track 450.8 -> 453.8 mm
Changed lines of the file:
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@@
 <attribute name="PROD_ID" value="RES-09883" x="21.95" y="32.65" size="1.778" layer="27" rot="R180" display="off"/>
+</element>
+<element name="C13" library="SparkFun-Capacitors" package="0603-CAP" value="10uF" x="4.2" y="27.6">
+<attribute name="PROD_ID" value="CAP-00810" x="4.2" y="27.6" size="1.778" layer="27" display="off"/>
 </element>
 </elements>
@@
 <wire x1="56.6" y1="26.2" x2="56.75" y2="26.05" width="0.254" layer="1"/>
 <wire x1="49.1" y1="23.556" x2="49.1" y2="25.8" width="0.254" layer="1"/>
+<contactref element="C13" pad="2"/>
+<wire x1="8.04" y1="27.538" x2="5.112" y2="27.538" width="0.3048" layer="1"/>
+<wire x1="5.112" y1="27.538" x2="5.05" y2="27.6" width="0.3048" layer="1"/>
 </signal>
 <signal name="N$58">
@@
 <wire x1="46.5" y1="52.5" x2="46.5" y2="59.75" width="0.254" layer="16"/>
 <via x="46.5" y="52.5" extent="1-16" drill="0.6096"/>
+<contactref element="C13" pad="1"/>
+<wire x1="3.27" y1="34.11" x2="3.27" y2="27.68" width="0.3048" layer="1"/>
+<wire x1="3.27" y1="27.68" x2="3.35" y2="27.6" width="0.3048" layer="1"/>
 </signal>
 <signal name="N$6">
