File: hardware/MSP430Geiger/MSP430Geiger.sch (EAGLE design)
At the start: 83 parts, among them IC1 LDO, IC2 MSP430, IC3 LM555D, IC4 LM555N, IC5 LM321MF, Q1 2N2222, Q2 MPSA42, Q3 2N2222, T1 DMN3024LSD, T2 2N2222(N.M)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

Commit message: edit
Parts:
- added C13: 10uF, SparkFun-Capacitors:0.1UF-25V(+80/-20%)(0603)
Connections:
- net GND: now also C13.2
- net VDD: now also C13.1
Changed lines of the file:
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@@
 <setting verticaltext="up"/>
 </settings>
-<grid distance="0.05" unitdist="inch" unit="inch" style="lines" multiple="1" display="no" altdistance="0.01" altunitdist="inch" altunit="inch"/>
+<grid distance="0.1" unitdist="inch" unit="inch" style="lines" multiple="1" display="no" altdistance="0.01" altunitdist="inch" altunit="inch"/>
 <layers>
 <layer number="1" name="Top" color="4" fill="1" visible="no" active="no"/>
@@
 <part name="GND28" library="SparkFun-Aesthetics" deviceset="GND" device=""/>
 <part name="R21" library="SparkFun-Resistors" deviceset="0.22OHM1/4W1%(0805)" device="" value="0"/>
+<part name="C13" library="SparkFun-Capacitors" deviceset="0.1UF-25V(+80/-20%)(0603)" device="" value="10uF"/>
 </parts>
 <sheets>
@@
 <instance part="GND28" gate="1" x="57.15" y="64.77"/>
 <instance part="R21" gate="G$1" x="180.34" y="71.12" rot="R180"/>
+<instance part="C13" gate="G$1" x="127" y="144.78"/>
 </instances>
 <busses>
@@
 <pinref part="C3" gate="G$1" pin="2"/>
 <wire x1="91.44" y1="142.24" x2="104.14" y2="142.24" width="0.1524" layer="91"/>
+<pinref part="C13" gate="G$1" pin="2"/>
+<wire x1="116.84" y1="142.24" x2="127" y2="142.24" width="0.1524" layer="91"/>
 </segment>
 <segment>
@@
 <pinref part="IC1" gate="G$1" pin="OUT@1"/>
 <wire x1="111.76" y1="147.32" x2="111.76" y2="149.86" width="0.1524" layer="91"/>
-</segment>
-<segment>
+<pinref part="C13" gate="G$1" pin="1"/>
+<wire x1="116.84" y1="149.86" x2="127" y2="149.86" width="0.1524" layer="91"/>
+</segment>
+<segment>
